Commit message: optical camera added

File: catkin_ws/src/my_robot/urdf/my_robot.xacro (robot description, xacro)
@@ -165,4 +165,9 @@
     </visual>
   </link>
+  <joint type="fixed" name="camera_optical_joint">
+    <origin xyz="0 0 0" rpy="-1.5707 0 -1.5707"/>
+    <child link="camera_link_optical"/>
+    <parent link="camera_link"/>
+  </joint>
   <joint type="fixed" name="hokuyo_joint">
     <origin xyz="0.15 0 0.1" rpy="0 0 0"/>
@@ -170,3 +175,5 @@
     <parent link="chassis"/>
   </joint>
+  <link name="camera_link_optical">
+  </link>
 </robot>

Commit message: fix urdf

File: catkin_ws/src/my_robot/urdf/my_robot.xacro (robot description, xacro)
@@ -118,5 +118,5 @@
     </visual>
   </link>
-  <link name="camera">
+  <link name="camera_link">
   <inertial>
     <mass value="0.1"/>
@@ -130,5 +130,5 @@
     </geometry>
   </collision>
-  <visual name='camera'>
+  <visual name='camera_link'>
     <origin xyz="0 0 0" rpy="0 0 0"/>
     <geometry>
@@ -139,5 +139,5 @@
   <joint type="fixed" name="camera_joint">
     <origin xyz="0.2 0 0" rpy="0 0 0"/>
-    <child link="camera"/>
+    <child link="camera_link"/>
     <parent link="chassis"/>
   </joint>

Commit message: base_footprint adapted

File: catkin_ws/src/my_robot/urdf/my_robot.xacro (robot description, xacro)
@@ -2,8 +2,8 @@
 <robot name="my_robot" xmlns:xacro="http://www.ros.org/wiki/xacro">
   <xacro:include filename="$(find my_robot)/urdf/my_robot.gazebo" />
-  <link name="robot_footprint"></link>
-  <joint name="robot_footprint_joint" type="fixed">
+  <link name="base_footprint"></link>
+  <joint name="base_footprint_joint" type="fixed">
     <origin xyz="0 0 0" rpy="0 0 0" />
-    <parent link="robot_footprint"/>
+    <parent link="base_footprint"/>
     <child link="chassis" />
   </joint>
